Commit message: Added husky_coal_navigation - unfinished

File: husky_coal_sim/husky_coal_description/urdf/husky_OS1-64_arch.urdf.xacro (robot description, xacro)
@@ -324,5 +324,5 @@
    <gazebo reference="box_link">
      <material>Gazebo/Red</material>
-     <transparency>0.9</transparency>
+     <transparency>0.6</transparency>
    </gazebo>
     <!--joint name="object_base_joint2" type="fixed">
@@ -433,5 +433,6 @@
     <!-- Add primary sensor arch/rail for OS1-64 LiDAR -->
     <xacro:sensor_arch prefix="OS1_" parent="base_link">
-      <origin xyz="0 0 0.25" rpy="$(arg laser_3d_rpy)"/>
+      <origin xyz="0.20 0 0.46" rpy="$(arg laser_3d_rpy)"/>
+<!--      <origin xyz="0 0 0.25" rpy="$(arg laser_3d_rpy)"/>  -->
     </xacro:sensor_arch>
     <!-- Ouster sensor links and fixed joints -->
